File: HW2/ME433/untitled2.sch (EAGLE design)
At the start: 22 parts, among them SW1 DIP-SLIDE-SWITCH(3P-11.6X4.0X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

Commit message: presmash
layout complete, presmash and prenaming
Parts:
- C3: device components:C-US050-030X075 -> components:C-US025-030X050
- PWR: value (none) -> RED
- U$1: value VOLTAGE_REGULATOR_MCP1702 -> VOLTAGE_REGULATOR_MCP1702TO92; device components:VOLTAGE_REGULATOR_MCP1702 -> components:VOLTAGE_REGULATOR_MCP1702TO92
- U$8: value PICKITROW -> PICKITROW5ROW; device components:PICKITROW -> components:PICKITROW5ROW
Connections:
- net A4: now also LED1.A; no longer LED.2
- net GND: now also LED.1; no longer LED1.C
- net N$1: now also LED.2, LED1.C; no longer LED.1, LED1.A
Other:
- moved on the sheet: LED, LED1
Changed lines of the file:
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@@
 <grid distance="0.1" unitdist="inch" unit="inch" style="lines" multiple="1" display="no" altdistance="0.01" altunitdist="inch" altunit="inch"/>
 <layers>
-<layer number="1" name="Top" color="4" fill="1" visible="no" active="no"/>
-<layer number="16" name="Bottom" color="1" fill="1" visible="no" active="no"/>
-<layer number="17" name="Pads" color="2" fill="1" visible="no" active="no"/>
-<layer number="18" name="Vias" color="2" fill="1" visible="no" active="no"/>
-<layer number="19" name="Unrouted" color="6" fill="1" visible="no" active="no"/>
-<layer number="20" name="Dimension" color="15" fill="1" visible="no" active="no"/>
-<layer number="21" name="tPlace" color="7" fill="1" visible="no" active="no"/>
-<layer number="22" name="bPlace" color="7" fill="1" visible="no" active="no"/>
-<layer number="23" name="tOrigins" color="15" fill="1" visible="no" active="no"/>
-<layer number="24" name="bOrigins" color="15" fill="1" visible="no" active="no"/>
-<layer number="25" name="tNames" color="7" fill="1" visible="no" active="no"/>
-<layer number="26" name="bNames" color="7" fill="1" visible="no" active="no"/>
-<layer number="27" name="tValues" color="7" fill="1" visible="no" active="no"/>
-<layer number="28" name="bValues" color="7" fill="1" visible="no" active="no"/>
+<layer number="1" name="Top" color="4" fill="1" visible="yes" active="no"/>
+<layer number="16" name="Bottom" color="1" fill="1" visible="yes" active="no"/>
+<layer number="17" name="Pads" color="2" fill="1" visible="yes" active="no"/>
+<layer number="18" name="Vias" color="2" fill="1" visible="yes" active="no"/>
+<layer number="19" name="Unrouted" color="6" fill="1" visible="yes" active="no"/>
+<layer number="20" name="Dimension" color="15" fill="1" visible="yes" active="no"/>
+<layer number="21" name="tPlace" color="7" fill="1" visible="yes" active="no"/>
+<layer number="22" name="bPlace" color="7" fill="1" visible="yes" active="no"/>
+<layer number="23" name="tOrigins" color="15" fill="1" visible="yes" active="no"/>
+<layer number="24" name="bOrigins" color="15" fill="1" visible="yes" active="no"/>
+<layer number="25" name="tNames" color="7" fill="1" visible="yes" active="no"/>
+<layer number="26" name="bNames" color="7" fill="1" visible="yes" active="no"/>
+<layer number="27" name="tValues" color="7" fill="1" visible="yes" active="no"/>
+<layer number="28" name="bValues" color="7" fill="1" visible="yes" active="no"/>
 <layer number="29" name="tStop" color="7" fill="3" visible="no" active="no"/>
 <layer number="30" name="bStop" color="7" fill="6" visible="no" active="no"/>
@@
 <layer number="35" name="tGlue" color="7" fill="4" visible="no" active="no"/>
 <layer number="36" name="bGlue" color="7" fill="5" visible="no" active="no"/>
-<layer number="37" name="tTest" color="7" fill="1" visible="no" active="no"/>
-<layer number="38" name="bTest" color="7" fill="1" visible="no" active="no"/>
+<layer number="37" name="tTest" color="7" fill="1" visible="yes" active="no"/>
+<layer number="38" name="bTest" color="7" fill="1" visible="yes" active="no"/>
 <layer number="39" name="tKeepout" color="4" fill="11" visible="no" active="no"/>
 <layer number="40" name="bKeepout" color="1" fill="11" visible="no" active="no"/>
@@
 <layer number="44" name="Drills" color="7" fill="1" visible="no" active="no"/>
 <layer number="45" name="Holes" color="7" fill="1" visible="no" active="no"/>
-<layer number="46" name="Milling" color="3" fill="1" visible="no" active="no"/>
-<layer number="47" name="Measures" color="7" fill="1" visible="no" active="no"/>
-<layer number="48" name="Document" color="7" fill="1" visible="no" active="no"/>
-<layer number="49" name="Reference" color="7" fill="1" visible="no" active="no"/>
-<layer number="50" name="dxf" color="7" fill="1" visible="no" active="no"/>
-<layer number="51" name="tDocu" color="7" fill="1" visible="no" active="no"/>
-<layer number="52" name="bDocu" color="7" fill="1" visible="no" active="no"/>
-<layer number="53" name="tGND_GNDA" color="7" fill="9" visible="no" active="no"/>
-<layer number="54" name="bGND_GNDA" color="1" fill="9" visible="no" active="no"/>
-<layer number="56" name="wert" color="7" fill="1" visible="no" active="no"/>
-<layer number="57" name="tCAD" color="7" fill="1" visible="no" active="no"/>
-<layer number="59" name="tCarbon" color="7" fill="1" visible="no" active="no"/>
-<layer number="60" name="bCarbon" color="7" fill="1" visible="no" active="no"/>
+<layer number="46" name="Milling" color="3" fill="1" visible="yes" active="no"/>
+<layer number="47" name="Measures" color="7" fill="1" visible="yes" active="no"/>
+<layer number="48" name="Document" color="7" fill="1" visible="yes" active="no"/>
+<layer number="49" name="Reference" color="7" fill="1" visible="yes" active="no"/>
+<layer number="50" name="dxf" color="7" fill="1" visible="yes" active="no"/>
+<layer number="51" name="tDocu" color="7" fill="1" visible="yes" active="no"/>
+<layer number="52" name="bDocu" color="7" fill="1" visible="yes" active="no"/>
+<layer number="53" name="tGND_GNDA" color="7" fill="9" visible="yes" active="no"/>
+<layer number="54" name="bGND_GNDA" color="1" fill="9" visible="yes" active="no"/>
+<layer number="56" name="wert" color="7" fill="1" visible="yes" active="no"/>
+<layer number="57" name="tCAD" color="7" fill="1" visible="yes" active="no"/>
+<layer number="59" name="tCarbon" color="7" fill="1" visible="yes" active="no"/>
+<layer number="60" name="bCarbon" color="7" fill="1" visible="yes" active="no"/>
 <layer number="90" name="Modules" color="5" fill="1" visible="yes" active="yes"/>
 <layer number="91" name="Nets" color="2" fill="1" visible="yes" active="yes"/>
@@
 </classes>
 <parts>
-<part name="U$1" library="components" deviceset="VOLTAGE_REGULATOR_MCP1702" device=""/>
+<part name="U$1" library="components" deviceset="VOLTAGE_REGULATOR_MCP1702" device="TO92" value="VOLTAGE_REGULATOR_MCP1702TO92"/>
 <part name="LED1" library="components" deviceset="TLLG4400" device=""/>
 <part name="BUTTON" library="components" deviceset="R-US_" device="0207/10" value="10k"/>
@@
 <part name="C1" library="components" deviceset="C-US" device="025-030X050" value="1uf"/>
 <part name="C2" library="components" deviceset="C-US" device="025-030X050" value="1uf"/>
-<part name="C3" library="components" deviceset="C-US" device="050-030X075" value=".1uf"/>
+<part name="C3" library="components" deviceset="C-US" device="025-030X050" value=".1uf"/>
 <part name="C4" library="components" deviceset="C-US" device="025-030X050" value=".1uf"/>
 <part name="C5" library="components" deviceset="C-US" device="025-030X050" value=".1uf"/>
@@
 <part name="+3V1" library="components" deviceset="+3V3" device=""/>
 <part name="GND1" library="components" deviceset="GND" device=""/>
-<part name="U$8" library="components" deviceset="PICKITROW" device=""/>
+<part name="U$8" library="components" deviceset="PICKITROW" device="5ROW" value="PICKITROW5ROW"/>
 <part name="SW1" library="components" deviceset="DIP-SLIDE-SWITCH(3P-11.6X4.0X5.4+2.0MM)" device="-EG1218"/>
 <part name="HEADER1" library="components" deviceset="M08" device="" value="1"/>
 <part name="HEADER2" library="components" deviceset="M08" device="" value="2"/>
 <part name="LED" library="components" deviceset="R-US_" device="0207/10" value="330"/>
-<part name="PWR" library="components" deviceset="LED" device="3MM"/>
+<part name="PWR" library="components" deviceset="LED" device="3MM" value="RED"/>
 <part name="RPWR" library="components" deviceset="R-US_" device="0207/10" value="330"/>
 </parts>
@@
 <instances>
 <instance part="U$1" gate="G$1" x="22.86" y="99.06"/>
-<instance part="LED1" gate="G$1" x="25.4" y="10.16"/>
+<instance part="LED1" gate="G$1" x="35.56" y="25.4"/>
 <instance part="BUTTON" gate="G$1" x="5.08" y="17.78"/>
 <instance part="MCLR" gate="G$1" x="35.56" y="58.42"/>
@@
 <instance part="HEADER1" gate="G$1" x="132.08" y="50.8"/>
 <instance part="HEADER2" gate="G$1" x="132.08" y="20.32"/>
-<instance part="LED" gate="G$1" x="35.56" y="20.32" rot="R90"/>
+<instance part="LED" gate="G$1" x="35.56" y="10.16" rot="R90"/>
 <instance part="PWR" gate="G$1" x="40.64" y="81.28" rot="R90"/>
 <instance part="RPWR" gate="G$1" x="58.42" y="81.28"/>
@@
 </segment>
 <segment>
-<pinref part="LED1" gate="G$1" pin="C"/>
-<wire x1="25.4" y1="5.08" x2="25.4" y2="2.54" width="0.1524" layer="91"/>
-<label x="25.4" y="0" size="1.778" layer="95"/>
-</segment>
-<segment>
 <pinref part="U$4" gate="G$1" pin="GND"/>
 <wire x1="63.5" y1="5.08" x2="78.74" y2="5.08" width="0.1524" layer="91"/>
@@
 <wire x1="63.5" y1="81.28" x2="68.58" y2="81.28" width="0.1524" layer="91"/>
 <label x="68.58" y="81.28" size="1.778" layer="95"/>
+</segment>
+<segment>
+<pinref part="LED" gate="G$1" pin="1"/>
+<wire x1="35.56" y1="5.08" x2="35.56" y2="2.54" width="0.1524" layer="91"/>
+<label x="33.02" y="2.54" size="1.778" layer="95"/>
 </segment>
 </net>
@@
 <pinref part="U$5" gate="G$1" pin="RA4"/>
 <wire x1="35.56" y1="30.48" x2="45.72" y2="30.48" width="0.1524" layer="91"/>
-<pinref part="LED" gate="G$1" pin="2"/>
-<wire x1="35.56" y1="30.48" x2="35.56" y2="25.4" width="0.1524" layer="91"/>
+<pinref part="LED1" gate="G$1" pin="A"/>
+<wire x1="35.56" y1="30.48" x2="35.56" y2="27.94" width="0.1524" layer="91"/>
 </segment>
 </net>
@@
 </segment>
 </net>
-<net name="N$1" class="0">
-<segment>
-<pinref part="LED1" gate="G$1" pin="A"/>
-<wire x1="25.4" y1="12.7" x2="35.56" y2="12.7" width="0.1524" layer="91"/>
-<pinref part="LED" gate="G$1" pin="1"/>
-<wire x1="35.56" y1="15.24" x2="35.56" y2="12.7" width="0.1524" layer="91"/>
-</segment>
-</net>
 <net name="N$2" class="0">
 <segment>
@@
 </segment>
 </net>
+<net name="N$1" class="0">
+<segment>
+<pinref part="LED1" gate="G$1" pin="C"/>
+<pinref part="LED" gate="G$1" pin="2"/>
+<wire x1="35.56" y1="20.32" x2="35.56" y2="15.24" width="0.1524" layer="91"/>
+</segment>
+</net>
