File: HW2/ME433/untitled3.brd (EAGLE design)
At the start: 50 x 50 mm, 22 parts

Commit message: Ready to be checked before order
updated voltage regulator package to TO-92 EBC and tweaked power traces
to avoid drill holes
Parts:
- U$1: value (none) -> VOLTAGE_REGULATOR_MCP1702; device components:TO92 -> components:TO92-EBC
- moved C1 4.19 mm to (42.2, 23.9), turned to 180 degrees
- moved U$1 3.77 mm to (47.0, 25.7)
- moved C2 2.50 mm to (42.2, 28.2), turned to 180 degrees
- moved SWITCH 1.55 mm to (47.9, 35.9)
Connections:
- net +3V3: now also U$1.E; no longer U$1.3
- net +5V: now also U$1.B; no longer U$1.2
- net GND: now also U$1.C; no longer U$1.1
Routing:
- net +5V: track 40.3 -> 47.4 mm
- net VBUS: track 6.59 -> 8.49 mm
Changed lines of the file:
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@@
 <setting verticaltext="up"/>
 </settings>
-<grid distance="0.8" unitdist="mil" unit="mil" style="lines" multiple="1" display="yes" altdistance="0.01" altunitdist="inch" altunit="inch"/>
+<grid distance="1.27" unitdist="mm" unit="mm" style="lines" multiple="1" display="yes" altdistance="0.01" altunitdist="inch" altunit="inch"/>
 <layers>
 <layer number="1" name="Top" color="4" fill="1" visible="yes" active="yes"/>
@@
 <wire x1="50" y1="50" x2="0" y2="50" width="0" layer="20"/>
 <wire x1="0" y1="50" x2="0" y2="0" width="0" layer="20"/>
-<text x="46.482" y="31.496" size="0.6096" layer="26" rot="MR0">+3v3</text>
-<text x="46.482" y="31.242" size="0.6096" layer="25" rot="R90">+5v</text>
+<text x="46.482" y="27.686" size="0.6096" layer="26" rot="MR0">+3v3</text>
+<text x="45.974" y="27.432" size="0.6096" layer="25" rot="R90">+5v</text>
 <polygon width="0.254" layer="25">
 <vertex x="1.27" y="2.54"/>
@@
 <attribute name="VALUE" x="33.2994" y="6.35" size="1.27" layer="27" ratio="10"/>
 </element>
-<element name="C1" library="components" package="C025-030X050" value="1uf" x="46.355" y="23.495" smashed="yes" rot="R270">
-<attribute name="VALUE" x="43.307" y="24.511" size="1.27" layer="27" ratio="10" rot="R270"/>
+<element name="C1" library="components" package="C025-030X050" value="1uf" x="42.179240625" y="23.891240625" smashed="yes" rot="R180">
+<attribute name="VALUE" x="43.195240625" y="22.113240625" size="1.27" layer="27" ratio="10" rot="R180"/>
 </element>
-<element name="C2" library="components" package="C025-030X050" value="1uf" x="43.18" y="30.48" smashed="yes" rot="R270">
-<attribute name="VALUE" x="40.132" y="33.782" size="1.27" layer="27" ratio="10" rot="R270"/>
+<element name="C2" library="components" package="C025-030X050" value="1uf" x="42.164" y="28.194" smashed="yes" rot="R180">
+<attribute name="VALUE" x="43.18" y="31.242" size="1.27" layer="27" ratio="10" rot="R180"/>
 </element>
 <element name="C3" library="components" package="C025-030X050" value=".1uf" x="2.54" y="38.735" smashed="yes">
@@
 <attribute name="VALUE" x="36.2966" y="18.415" size="1.27" layer="27" ratio="10" rot="R180"/>
 </element>
-<element name="SWITCH" library="components" package="SW3-2.5-11.6X4.0X5.4+2.0MM" value="" x="47.625" y="37.465" smashed="yes" rot="R270">
-<attribute name="NAME" x="48.641" y="39.37" size="0.889" layer="25" ratio="11" rot="R270"/>
-<attribute name="VALUE" x="44.45" y="39.878" size="0.635" layer="27" ratio="11" rot="R270"/>
-</element>
-<element name="U$1" library="components" package="TO92" value="" x="48.26" y="29.21" smashed="yes" rot="R90">
-<attribute name="VALUE" x="49.53" y="32.385" size="1.27" layer="27" ratio="10" rot="R90"/>
+<element name="SWITCH" library="components" package="SW3-2.5-11.6X4.0X5.4+2.0MM" value="" x="47.879" y="35.941" smashed="yes" rot="R270">
+<attribute name="NAME" x="48.895" y="37.846" size="0.889" layer="25" ratio="11" rot="R270"/>
+<attribute name="VALUE" x="44.704" y="38.354" size="0.635" layer="27" ratio="11" rot="R270"/>
 </element>
+<element name="U$1" library="components" package="TO92-EBC" value="VOLTAGE_REGULATOR_MCP1702" x="47.01031875" y="25.654" smashed="yes" rot="R90"/>
 <element name="C6" library="components" package="C025-040X050POL" value="10uf" x="21.59" y="41.91" smashed="yes" rot="R90">
 <attribute name="VALUE" x="19.177" y="40.386" size="1.27" layer="27" ratio="10" rot="R90"/>
@@
 <signal name="GND">
 <contactref element="U$8" pad="3"/>
-<contactref element="U$1" pad="1"/>
+<contactref element="U$1" pad="C"/>
 <contactref element="U$5" pad="8"/>
 <contactref element="U$5" pad="27"/>
@@
 <signal name="+3V3">
 <contactref element="U$8" pad="2"/>
-<contactref element="U$1" pad="3"/>
+<contactref element="U$1" pad="E"/>
 <contactref element="PWR" pad="A"/>
 <contactref element="U$5" pad="13"/>
@@
 <contactref element="C3" pad="1"/>
 <wire x1="1.27" y1="38.735" x2="1.27" y2="35.56" width="0.4064" layer="1"/>
-<wire x1="40.005" y1="30.48" x2="33.655" y2="30.48" width="1.27" layer="16"/>
+<wire x1="38.735" y1="30.48" x2="33.655" y2="30.48" width="1.27" layer="16"/>
 <wire x1="33.655" y1="30.48" x2="31.75" y2="30.48" width="1.27" layer="16"/>
 <wire x1="31.75" y1="27.94" x2="31.75" y2="28.575" width="1.27" layer="16"/>
@@
 <wire x1="27.94" y1="34.29" x2="31.75" y2="30.48" width="0.8128" layer="1"/>
 <via x="31.75" y="30.48" extent="1-16" drill="0.6"/>
-<via x="40.005" y="30.48" extent="1-16" drill="0.6"/>
-<wire x1="31.75" y1="21.59" x2="39.37" y2="21.59" width="1.27" layer="16"/>
-<wire x1="40.005" y1="30.48" x2="40.005" y2="22.225" width="1.27" layer="1"/>
-<wire x1="40.005" y1="22.225" x2="39.37" y2="21.59" width="1.27" layer="1"/>
-<via x="39.37" y="21.59" extent="1-16" drill="0.6"/>
+<via x="38.735" y="30.48" extent="1-16" drill="0.6"/>
+<wire x1="31.75" y1="21.59" x2="38.1" y2="21.59" width="1.27" layer="16"/>
+<wire x1="38.735" y1="30.48" x2="38.735" y2="23.495" width="1.27" layer="1"/>
+<wire x1="38.735" y1="23.495" x2="38.1" y2="21.59" width="1.27" layer="1"/>
+<via x="38.1" y="21.59" extent="1-16" drill="0.6"/>
 <wire x1="48.26" y1="17.78" x2="48.26" y2="19.05" width="0.4064" layer="16"/>
 <wire x1="48.26" y1="19.05" x2="47.625" y2="19.685" width="0.4064" layer="16"/>
 <wire x1="47.625" y1="19.685" x2="41.275" y2="19.685" width="0.4064" layer="16"/>
-<wire x1="41.275" y1="19.685" x2="39.37" y2="21.59" width="0.4064" layer="16"/>
+<wire x1="41.275" y1="19.685" x2="38.1" y2="21.59" width="0.4064" layer="16"/>
 <wire x1="30.48" y1="6.985" x2="30.48" y2="8.89" width="0.4064" layer="1"/>
 <wire x1="30.48" y1="8.89" x2="31.75" y2="10.16" width="0.4064" layer="1"/>
@@
 <wire x1="5.842" y1="30.48" x2="1.27" y2="35.052" width="1.27" layer="1"/>
 <wire x1="1.27" y1="35.052" x2="1.27" y2="35.56" width="1.27" layer="1"/>
-<wire x1="48.26" y1="30.48" x2="46.99" y2="31.75" width="1.27" layer="16"/>
-<wire x1="46.99" y1="31.75" x2="43.18" y2="31.75" width="1.27" layer="16"/>
-<wire x1="40.005" y1="30.48" x2="41.91" y2="30.48" width="1.27" layer="16"/>
-<wire x1="41.91" y1="30.48" x2="43.18" y2="31.75" width="1.27" layer="16"/>
+<wire x1="48.28031875" y1="28.194" x2="43.434" y2="28.194" width="1.27" layer="16"/>
+<wire x1="43.434" y1="28.194" x2="43.434" y2="28.448" width="1.27" layer="16"/>
+<wire x1="43.434" y1="28.448" x2="41.402" y2="30.48" width="1.27" layer="16"/>
+<wire x1="41.402" y1="30.48" x2="38.735" y2="30.48" width="1.27" layer="16"/>
 </signal>
 <signal name="+5V">
 <contactref element="U$5" pad="15"/>
-<contactref element="U$1" pad="2"/>
+<contactref element="U$1" pad="B"/>
 <contactref element="C1" pad="1"/>
 <contactref element="SWITCH" pad="RIGHT"/>
 <contactref element="HEADER2" pad="7"/>
-<wire x1="47.625" y1="35.465" x2="47.53" y2="35.465" width="1.27" layer="1"/>
-<wire x1="47.53" y1="35.465" x2="46.355" y2="33.655" width="1.27" layer="1"/>
-<wire x1="46.355" y1="33.655" x2="46.355" y2="29.21" width="1.27" layer="1"/>
-<wire x1="46.355" y1="29.21" x2="46.355" y2="24.765" width="1.27" layer="1"/>
 <wire x1="34.29" y1="35.56" x2="36.83" y2="35.56" width="1.27" layer="16"/>
-<wire x1="36.83" y1="35.56" x2="47.085" y2="35.56" width="1.27" layer="16"/>
-<wire x1="47.085" y1="35.56" x2="47.625" y2="35.465" width="1.27" layer="16"/>
 <wire x1="36.83" y1="39.37" x2="36.83" y2="35.56" width="1.27" layer="1"/>
 <via x="36.83" y="35.56" extent="1-16" drill="0.6"/>
 <wire x1="30.734" y1="48.895" x2="30.734" y2="45.466" width="1.27" layer="1"/>
 <wire x1="30.734" y1="45.466" x2="36.83" y2="39.37" width="1.27" layer="1"/>
+<wire x1="47.879" y1="33.941" x2="38.449" y2="33.941" width="1.27" layer="16"/>
+<wire x1="38.449" y1="33.941" x2="36.83" y2="35.56" width="1.27" layer="16"/>
+<wire x1="48.28031875" y1="25.654" x2="45.212" y2="25.654" width="1.27" layer="16"/>
+<wire x1="45.212" y1="25.654" x2="43.449240625" y2="23.891240625" width="1.27" layer="16"/>
+<wire x1="48.28031875" y1="25.654" x2="46.736" y2="25.654" width="1.27" layer="1"/>
+<wire x1="46.736" y1="25.654" x2="45.72" y2="26.67" width="1.27" layer="1"/>
+<wire x1="45.72" y1="26.67" x2="45.72" y2="32.766" width="1.27" layer="1"/>
+<wire x1="47.879" y1="33.941" x2="46.895" y2="33.941" width="1.27" layer="1"/>
+<wire x1="46.895" y1="33.941" x2="45.72" y2="32.766" width="1.27" layer="1"/>
 </signal>
 <signal name="MCLR">
@@
 <contactref element="SWITCH" pad="C"/>
 <contactref element="U$4" pad="VBUS"/>
-<wire x1="46.05" y1="43.16" x2="46.05" y2="38.405" width="1.27" layer="1"/>
-<wire x1="46.05" y1="38.405" x2="47.625" y2="37.465" width="1.27" layer="1"/>
+<wire x1="47.879" y1="35.941" x2="47.117" y2="35.941" width="0.8128" layer="1"/>
+<wire x1="47.117" y1="35.941" x2="45.974" y2="37.084" width="0.8128" layer="1"/>
+<wire x1="45.974" y1="37.084" x2="45.974" y2="43.084" width="0.8128" layer="1"/>
+<wire x1="45.974" y1="43.084" x2="46.05" y2="43.16" width="0.8128" layer="1"/>
 </signal>
 <signal name="A0">

Commit message: Ready to checked before ordering v3
some more board tweaks, removed redundant via
Routing:
- net USBD+: vias 2 -> 0
Changed lines of the file:
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@@
 <contactref element="U$5" pad="21"/>
 <contactref element="U$4" pad="D+"/>
-<wire x1="44.45" y1="43.16" x2="44.45" y2="43.18" width="0.4064" layer="1"/>
-<wire x1="44.45" y1="43.16" x2="44.45" y2="40.64" width="0.4064" layer="1"/>
-<wire x1="44.45" y1="40.64" x2="41.91" y2="38.1" width="0.4064" layer="1"/>
-<via x="41.91" y="38.1" extent="1-16" drill="0.6"/>
 <wire x1="41.91" y1="38.1" x2="20.32" y2="38.1" width="0.4064" layer="16"/>
 <wire x1="20.32" y1="38.1" x2="19.05" y2="36.83" width="0.4064" layer="16"/>
 <wire x1="19.05" y1="36.83" x2="19.05" y2="35.56" width="0.4064" layer="16"/>
-<via x="44.45" y="40.64" extent="1-16" drill="0.6"/>
+<wire x1="41.91" y1="38.1" x2="44.45" y2="40.64" width="0.4064" layer="16"/>
+<wire x1="44.45" y1="40.64" x2="44.45" y2="43.16" width="0.4064" layer="16"/>
 </signal>
 <signal name="USBD-">
